Commit message: first by mcqueen

File: urdf/livox_mid360.xacro (robot description, xacro)
@@ -22,5 +22,5 @@
         <update_rate>${update_rate}</update_rate>
         <!-- This ray plgin is only for visualization. -->
-        <plugin name="gazebo_ros_laser_controller" filename="liblivox_laser_simulation.so">
+        <plugin name="lidar" filename="liblivox_laser_simulation.so">
 			<ray>
 			  <scan>
@@ -53,4 +53,5 @@
 		  <downsample>${downsample}</downsample>
 		  <csv_file_name>package://livox_laser_simulation/scan_mode/mid360.csv</csv_file_name>
+          <publish_pointcloud_type>1</publish_pointcloud_type>
 		  <ros_topic>${ros_topic}</ros_topic>
         </plugin>
@@ -58,11 +59,11 @@
     </gazebo>
   </xacro:macro>
-  <xacro:macro name="Livox_Mid40" params="visualize:=True name:=livox">
+  <xacro:macro name="Livox_Mid360" params="visualize:=True name:=livox">
     <link name="${name}_base">
       <xacro:null_inertial/>
       <visual>
-        <origin xyz="0.00 0 0.0" rpy="0 0 0"/>
+        <origin xyz="0 0 0" rpy="0 0 0"/>
         <geometry>
-          <mesh filename="package://livox_laser_simulation/meshes/livox_mid40.dae">
+          <mesh filename="package://livox_laser_simulation/meshes/livox_mid360.dae">
           </mesh>
         </geometry>
@@ -70,5 +71,5 @@
       <collision>
 		  <origin xyz="0 0 0" rpy="0 0 0" /> <geometry> <mesh
-		  filename="package://livox_laser_simulation/meshes/livox_mid40.dae">
+		  filename="package://livox_laser_simulation/meshes/livox_mid360.dae">
 		  </mesh> </geometry>
       </collision>
@@ -80,10 +81,8 @@
       <parent link="${name}_base"/>
       <child link="${name}"/>
-      <origin rpy="0 0 0" xyz="0.0 1.0 0.2"/>
+      <origin rpy="0 0 0" xyz="0 0 0"/>
     </joint>
     <xacro:Livox_Mid_gazebo_sensor name="${name}" visualize="${visualize}"/>
   </xacro:macro>
-    <xacro:Livox_Mid40 name="livox"/>
-  <xacro:include filename="$(find livox_laser_simulation)/urdf/standardrobots_oasis300.xacro"/>
-  <xacro:link_oasis name="oasis"/>
+    <xacro:Livox_Mid360 name="livox"/>
 </robot>
